Commit message: changed material name

File: urdf/materials.xacro (robot description, xacro)
@@ -4,5 +4,5 @@
   <color rgba="0.700 0.700 0.700 1.000"/>
 </material>
-<material name="shit">
+<material name="blue">
     <!-- <ambient>0.0 0.0 1.0 1</ambient>
     <diffuse>0.0 0.0 1.0 1</diffuse>

File: urdf/minimal_robot.xacro (robot description, xacro)
@@ -26,5 +26,5 @@
         <mesh filename="package://rebob_sim_description/meshes/base_link.stl" scale="0.001 0.001 0.001"/>
       </geometry> -->
-      <material name="shit"/>
+      <material name="blue"/>
     </visual>
     <collision>
